File: Spinne_Werkstatt.kicad_sch (KiCad schematic)
At the start: 15 parts, among them J1 Conn_01x02_Pin, J3 Conn_01x03_Pin, Q1 BSS138, Q2 BSS138, U2 CH340C, U4 ESP32-WROOM-32

Commit message: added esp32 wroom 32UE
Parts:
- removed U4: ESP32-WROOM-32, bulme_footprints:ESP32-WROOM-32D, symbol RF_Module:ESP32-WROOM-32
- added U1: ESP32-WROOM-32UE, RF_Module:ESP32-WROOM-32UE, symbol RF_Module:ESP32-WROOM-32UE
Connections:
- net +3V3: now also U1.2 (VDD)
- net ESP32_EN: now also U1.3 (EN)
- net ESP32_IO0: now also U1.25 (IO0)
- net ESP32_RX: now also U1.34 (RXD0/IO3)
- net ESP32_TX: now also U1.35 (TXD0/IO1)
- net GND: now also U1.1 (GND), U1.15 (GND), U1.38 (GND), U1.39 (GND)
- net SCL: now also U1.36 (IO22)
- net SDA: now also U1.33 (IO21)
- net pin10: now also U1.10 (IO25)
- net pin11: now also U1.11 (IO26)
- net pin12: now also U1.12 (IO27)
- net pin13: now also U1.13 (IO14)
- net pin14: now also U1.14 (IO12)
- net pin16: now also U1.16 (IO13)
- net pin23: now also U1.23 (IO15)
- net pin24: now also U1.24 (IO2)
- net pin26: now also U1.26 (IO4)
- net pin27: now also U1.27 (IO16)
- net pin28: now also U1.28 (IO17)
- net pin29: now also U1.29 (IO5)
- net pin30: now also U1.30 (IO18)
- net pin31: now also U1.31 (IO19)
- net pin37: now also U1.37 (IO23)
- net pin4: now also U1.4 (SENSOR_VP)
- net pin5: now also U1.5 (SENSOR_VN)
- net pin6: now also U1.6 (IO34)
- net pin7: now also U1.7 (IO35)
- net pin8: now also U1.8 (IO32)
- net pin9: now also U1.9 (IO33)
Changed lines of the file:
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@@
+	)
+	(symbol
+		(lib_id "RF_Module:ESP32-WROOM-32UE")
+		(at 54.61 204.47 0)
+		(unit 1)
+		(exclude_from_sim no)
+		(in_bom yes)
+		(on_board yes)
+		(dnp no)
+		(fields_autoplaced yes)
+		(property "Reference" "U1"
+			(at 56.7533 166.37 0)
+			(effects
+				(font
+					(size 1.27 1.27)
+				)
+				(justify left)
+			)
+		)
+		(property "Value" "ESP32-WROOM-32UE"
+			(at 56.7533 168.91 0)
+			(effects
+				(font
+					(size 1.27 1.27)
+				)
+				(justify left)
+			)
+		)
+		(property "Footprint" "RF_Module:ESP32-WROOM-32UE"
+			(at 71.12 238.76 0)
+			(effects
+				(font
+					(size 1.27 1.27)
+				)
+				(hide yes)
+			)
+		)
+		(property "Datasheet" "https://www.espressif.com/sites/default/files/documentation/esp32-wroom-32e_esp32-wroom-32ue_datasheet_en.pdf"
+			(at 54.61 204.47 0)
+			(effects
+				(font
+					(size 1.27 1.27)
+				)
+				(hide yes)
+			)
+		)
+		(property "Description" "RF Module, ESP32-D0WD-V3 SoC, without PSRAM, Wi-Fi 802.11b/g/n, Bluetooth, BLE, 32-bit, 2.7-3.6V, external antenna, SMD"
+			(at 54.61 204.47 0)
+			(effects
+				(font
+					(size 1.27 1.27)
+				)
+				(hide yes)
+			)
+		)
+		(pin "31"
+		)
+		(pin "16"
+		)
+		(pin "21"
+		)
+		(pin "20"
+		)
+		(pin "25"
+		)
+		(pin "18"
+		)
+		(pin "37"
+		)
+		(pin "36"
+		)
+		(pin "12"
+		)
+		(pin "15"
+		)
+		(pin "24"
+		)
+		(pin "26"
+		)
+		(pin "6"
+		)
+		(pin "39"
+		)
+		(pin "27"
+		)
+		(pin "28"
+		)
+		(pin "1"
+		)
+		(pin "2"
+		)
+		(pin "14"
+		)
+		(pin "3"
+		)
+		(pin "30"
+		)
+		(pin "32"
+		)
+		(pin "38"
+		)
+		(pin "33"
+		)
+		(pin "19"
+		)
+		(pin "13"
+		)
+		(pin "8"
+		)
+		(pin "22"
+		)
+		(pin "7"
+		)
+		(pin "9"
+		)
+		(pin "17"
+		)
+		(pin "29"
+		)
+		(pin "10"
+		)
+		(pin "34"
+		)
+		(pin "35"
+		)
+		(pin "11"
+		)
+		(pin "5"
+		)
+		(pin "4"
+		)
+		(pin "23"
+		)
+		(instances
+			(project ""
+				(path "/63f5a8da-c9e8-4b26-9a17-2dbcdac59688"
+					(reference "U1")
+					(unit 1)
+				)
+			)
+		)
 	)
 	(symbol
@@
 					(unit 1)
 				)
-			)
-		)
-	)
-	(symbol
-		(lib_id "RF_Module:ESP32-WROOM-32")
-		(at 54.61 204.47 0)
-		(unit 1)
-		(exclude_from_sim no)
-		(in_bom yes)
-		(on_board yes)
-		(dnp no)
-		(fields_autoplaced yes)
-		(property "Reference" "U4"
-			(at 56.7533 166.37 0)
-			(effects
-				(font
-					(size 1.27 1.27)
-				)
-				(justify left)
-			)
-		)
-		(property "Value" "ESP32-WROOM-32"
-			(at 56.7533 168.91 0)
-			(effects
-				(font
-					(size 1.27 1.27)
-				)
-				(justify left)
-			)
-		)
-		(property "Footprint" "bulme_footprints:ESP32-WROOM-32D"
-			(at 54.61 242.57 0)
-			(effects
-				(font
-					(size 1.27 1.27)
-				)
-				(hide yes)
-			)
-		)
-		(property "Datasheet" "https://www.espressif.com/sites/default/files/documentation/esp32-wroom-32_datasheet_en.pdf"
-			(at 46.99 203.2 0)
-			(effects
-				(font
-					(size 1.27 1.27)
-				)
-				(hide yes)
-			)
-		)
-		(property "Description" "RF Module, ESP32-D0WDQ6 SoC, Wi-Fi 802.11b/g/n, Bluetooth, BLE, 32-bit, 2.7-3.6V, onboard antenna, SMD"
-			(at 54.61 204.47 0)
-			(effects
-				(font
-					(size 1.27 1.27)
-				)
-				(hide yes)
-			)
-		)
-		(pin "31"
-		)
-		(pin "32"
-		)
-		(pin "18"
-		)
-		(pin "19"
-		)
-		(pin "21"
-		)
-		(pin "33"
-		)
-		(pin "39"
-		)
-		(pin "13"
-		)
-		(pin "11"
-		)
-		(pin "8"
-		)
-		(pin "2"
-		)
-		(pin "16"
-		)
-		(pin "17"
-		)
-		(pin "15"
-		)
-		(pin "9"
-		)
-		(pin "12"
-		)
-		(pin "1"
-		)
-		(pin "10"
-		)
-		(pin "14"
-		)
-		(pin "28"
-		)
-		(pin "5"
-		)
-		(pin "30"
-		)
-		(pin "24"
-		)
-		(pin "22"
-		)
-		(pin "7"
-		)
-		(pin "37"
-		)
-		(pin "38"
-		)
-		(pin "4"
-		)
-		(pin "20"
-		)
-		(pin "35"
-		)
-		(pin "26"
-		)
-		(pin "3"
-		)
-		(pin "25"
-		)
-		(pin "36"
-		)
-		(pin "23"
-		)
-		(pin "34"
-		)
-		(pin "27"
-		)
-		(pin "6"
-		)
-		(pin "29"
-		)
-		(instances
-			(project "Spinne_Werkstatt"
-				(path "/63f5a8da-c9e8-4b26-9a17-2dbcdac59688"
-					(reference "U4")
-					(unit 1)
-				)
