File: _autosave-Spinne_Werkstatt.kicad_sch (KiCad schematic)
At the start: 17 parts, among them J1 Conn_01x02_Pin, J3 Conn_01x03_Pin, Q1 BSS138, Q2 BSS138, U1 ESP32-WROOM-32UE, U2 CH340C

Commit message: nearly finished, not perfect but ok
Parts:
- renumbered ESP_EN_R to ESP_EN_R1
Changed lines of the file:
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@@
 		(dnp no)
 		(fields_autoplaced yes)
-		(property "Reference" "ESP_EN_R"
+		(property "Reference" "ESP_EN_R1"
 			(at 379.73 46.9899 0)
 			(effects
@@
 			(project ""
 				(path "/63f5a8da-c9e8-4b26-9a17-2dbcdac59688"
-					(reference "ESP_EN_R")
+					(reference "ESP_EN_R1")
 					(unit 1)
 				)
